File: kicad/io.kicad_sch (KiCad schematic)
At the start: 26 parts, among them J2 DB9 female, U6 74HC138, U7 W65C22N6TPG-14, U8 W65C51N, U9 MAX232N, X2 1.8432MHz

Commit message: Schematic rev 2: prepare the design for a 4-layer PCB
Keeps the breadboard's parts and logic and adds what a board needs.

- RDY, NMI, ABORT and BE get 3.3k pull-ups instead of hard ties to +5V
  (RDY is bidirectional; WAI drives it low).
- VDA and VPA go to GAL pins 11 and 13. New pld/decode03.pld (816DEC03)
  qualifies /IOSEL with VDA + VPA so internal-operation cycles cannot
  read and clear ACIA/VIA registers. decode.pld (816DEC02) stays for the
  breadboard.
- PHI2 from the GAL can be routed through a 74ACT08 buffer via JP2
  (default: direct, as built). Timing in decode03.pld NOTE 8.
- Clock source jumper JP1 and external clock header J5.
- New power sheet: USB-C (power only) or bench terminal via JP4, power
  switch, polyfuse, P-FET reverse-polarity protection, 47uF bulk, power
  LED, and 100nF decoupling per package.
- New expansion sheet: 2x30 bus header (address, latched bank byte,
  data, control, spare I/O slots), 2x12 VIA header, LED disconnect
  jumper, test points, mounting holes.
- Footprints on every part; socket footprints for all ICs.

ERC (KiCad 9.0.4 kicad-cli): 0 errors, 0 warnings. Both PLD files
assemble with Galette 0.3.0.

Co-Authored-By: Claude Opus 5.5 <noreply@anthropic.com>
Claude-Session: https://claude.ai/code/session_01WF6ESyzfg6uQED2DRD2W4Z
Parts:
- C2, C3, C4, C5: footprint (none) -> Capacitor_THT:CP_Radial_D5.0mm_P2.00mm
- D1, D2, D3, D4, D5, D6, D7, D8: footprint (none) -> LED_THT:LED_D3.0mm
- J2: footprint (none) -> Connector_Dsub:DSUB-9_Socket_Horizontal_P2.77x2.84mm_EdgePinOffset7.70mm_Housed_MountingHolesOffset9.12mm
- R10, R3, R4, R5, R6, R7, R8, R9: footprint (none) -> Resistor_THT:R_Axial_DIN0207_L6.3mm_D2.5mm_P7.62mm_Horizontal
- U6, U9: footprint Package_DIP:DIP-16_W7.62mm -> Package_DIP:DIP-16_W7.62mm_Socket
- U7: footprint Package_DIP:DIP-40_W15.24mm -> Package_DIP:DIP-40_W15.24mm_Socket
- U8: footprint Package_DIP:DIP-28_W15.24mm -> Package_DIP:DIP-28_W15.24mm_Socket
Connections:
- net GND: no longer R10.2, R3.2, R4.2, R5.2, R6.2, R7.2, R8.2, R9.2
- net ~{IO5}: now reaches U6.10 (~{Y5})
- net ~{IO3}: now reaches U6.12 (~{Y3})
- net ~{IO2}: now reaches U6.13 (~{Y2})
- net ~{IO1}: now reaches U6.14 (~{Y1})
- net ~{IO7}: now reaches U6.7 (~{Y7})
- net ~{IO6}: now reaches U6.9 (~{Y6})
- net CB1: now reaches U7.18 (CB1)
- net CB2: now reaches U7.19 (CB2)
- net PA0: now reaches U7.2 (PA0)
- net PA1: now reaches U7.3 (PA1)
- net CA2: now reaches U7.39 (CA2)
- net PA2: now reaches U7.4 (PA2)
- net CA1: now reaches U7.40 (CA1)
- net PA3: now reaches U7.5 (PA3)
- net PA4: now reaches U7.6 (PA4)
- net PA5: now reaches U7.7 (PA5)
- net PA6: now reaches U7.8 (PA6)
- net PA7: now reaches U7.9 (PA7)
- new net LED_GND: R10.2, R3.2, R4.2, R5.2, R6.2, R7.2, R8.2, R9.2
- no-connect marks 28 -> 10
Other:
- note added: "I/O window $00:6000-$00:7FFF, 8 x 1 KB slots on A12:A11:A10 ~{Y0} $6000 VIA ~{Y4} $7000 ACIA ~{Y1} $6400 ~{Y2} $6800 ~{Y3} $6C00 ~{Y5} $7400 ~{Y6} $7800 ~{Y7} $7C00 (to the expansion header as ~{IOn}) ~{E1} (pin 5) is the reserved PHI2 hook: tie to ~{PHI2} to qualify the selects later (decode.pld NOTE 2). E2 (pin 6) is the active-high enable - it must be high."
- note added: "Port A, Port B, CA1, CA2, CB1 and CB2 go to the VIA header J4 (expansion sheet). IRQB is open drain on the W65C22N: wired straight to ~{IRQ} (pull-up R2, CPU sheet)."
- note added: "Port B LEDs: PBn -> LED -> resistor -> LED_GND. LED_GND reaches GND through JP3 (expansion sheet); pull the jumper to free Port B for the header. R3-R10: 1k."
- note removed: "I/O window $00:6000-$00:7FFF, 8 x 1 KB slots on A12:A11:A10 ~{Y0} $6000 VIA ~{Y4} $7000 ACIA ~{Y1} $6400 ~{Y2} $6800 ~{Y3} $6C00 ~{Y5} $7400 ~{Y6} $7800 ~{Y7} $7C00 (unallocated, not connected) ~{E1} (pin 5) is the reserved PHI2 hook: tie to ~{PHI2} to qualify the selects later (decode.pld NOTE 2). E2 (pin 6) is the active-high enable - it must be high."
- note removed: "Port A, CA1, CA2, CB1, CB2 not connected. IRQB is open drain on the W65C22N: wired straight to ~{IRQ} (pull-up R2, CPU sheet)."
- note removed: "Port B LEDs: PBn -> LED -> resistor -> GND. R3-R10: 1k (measured)."
