File: kicad/io.kicad_sch (KiCad schematic)
At the start: 11 parts, among them J2 PORT A, J3 PORT B, J4 SERIAL (TTL), U7 74HC138, U8 W65C22, U9 W65C51N, Y1 1.8432MHz

Commit message: Update KiCad schematic to match the build as wired
- Remove video RAM (future expansion); GAL ~{VRAMCE} is NC and
  ~{WEGATE} goes only to the RAM
- VIA is a W65C22N6TPG-14: IRQB wired directly to ~{IRQ} (no diode)
- RDY and ~{NMI} tied directly to +5V; only reset and ~{IRQ} pull-ups
- ACIA clocked by a 1.8432 MHz DIP-8 oscillator on XTLI (EN high)
- Serial through a MAX232N to a female DB9 (pins 2, 3, 8, 5)
- VIA Port B drives eight LEDs with series resistors; Port A, CA/CB NC
- Drop per-chip decoupling; single 0.1uF electrolytic at the supply
- Unknown resistor values shown as '?'
- Update kicad/README.md and README.md accordingly

Co-Authored-By: Claude Opus 5.5 <noreply@anthropic.com>
Claude-Session: https://claude.ai/code/session_01GgTWzZQQJPzWrEMiSDZH6j
Parts:
- removed C10, C8: 100nF, symbol be6502:C
- removed D1: BAT85, symbol be6502:D_Schottky
- removed J3: PORT B, symbol be6502:Conn_01x10
- removed U9: W65C51N, Package_DIP:DIP-28_W15.24mm, symbol be6502:W65C51N
- added C4, C5: 1uF, symbol be6502:C_Polarized
- added D1, D2, D3, D4, D5, D6, D7, D8: LED, symbol be6502:LED
- added R10, R3, R4, R5, R6, R7, R8: ?, symbol be6502:R
- added U6: 74HC138, Package_DIP:DIP-16_W7.62mm, symbol be6502:74HC138
- added U7: W65C22N6TPG-14, Package_DIP:DIP-40_W15.24mm, symbol be6502:W65C22
- added U9: MAX232N, Package_DIP:DIP-16_W7.62mm, symbol be6502:MAX232
- C2: renamed from Y1; value 1.8432MHz -> 1uF; symbol be6502:Crystal -> be6502:C_Polarized
- C3: renamed from J4; value SERIAL (TTL) -> 1uF; symbol be6502:Conn_01x06 -> be6502:C_Polarized
- J2: renamed from C9; value 100nF -> DB9 female; symbol be6502:C -> be6502:DE9_Receptacle
- R9: renamed from U7; value 74HC138 -> ?; symbol be6502:74HC138 -> be6502:R
- U8: value W65C22 -> W65C51N; footprint Package_DIP:DIP-40_W15.24mm -> Package_DIP:DIP-28_W15.24mm; symbol be6502:W65C22 -> be6502:W65C51N
- X2: renamed from J2; value PORT A -> 1.8432MHz; footprint (none) -> Oscillator:Oscillator_DIP-8; symbol be6502:Conn_01x10 -> be6502:OSC_DIP8
Connections:
- net CB1 is gone; now on net D0: U8.18 (D0)
- net CB2 is gone; now on net D1: U8.19 (D1)
- net PA0 is gone; now on net VCC: U8.2 (CS0), X2.1 (EN)
- net ~{VIA_IRQ} is gone; now on net D3: U8.21 (D3)
- net A0: now also U8.13 (RS0), U7.38 (RS0); no longer U8.38 (RS0)
- net A1: now also U8.14 (RS1), U7.37 (RS1); no longer U8.37 (RS1)
- net A10: now also U6.1 (A0); no longer R9.1 (A0)
- net A11: now also U6.2 (A1); no longer R9.2 (A1)
- net A12: now also U6.3 (A2); no longer R9.3 (A2)
- net A2: now also U7.36 (RS2); no longer U8.36 (RS2)
- net A3: now also U7.35 (RS3); no longer U8.35 (RS3)
- net ACIA_RXD: now also U8.12 (RxD), U9.12 (R1OUT); no longer C3.4 (Pin_4)
- net ACIA_TXD: now also U8.10 (TxD), U9.11 (T1IN); no longer C3.5 (Pin_5)
- net D0: now also U7.33 (D0); no longer U8.33 (D0)
- net D1: now also U7.32 (D1); no longer U8.32 (D1)
- net D2: now also U8.20 (D2), U7.31 (D2); no longer U8.31 (D2)
- net D3: now also U7.30 (D3); no longer U8.30 (D3)
- net D4: now also U8.22 (D4), U7.29 (D4); no longer U8.29 (D4)
- net D5: now also U8.23 (D5), U7.28 (D5); no longer U8.28 (D5)
- net D6: now also U8.24 (D6), U7.27 (D6); no longer U8.27 (D6)
- net D7: now also U8.25 (D7), U7.26 (D7); no longer U8.26 (D7)
- net GND: now also J2.5, R9.2, U8.16 (~{DCD}), U8.17 (~{DSR}), U8.9 (~{CTS}), X2.4 (GND), C4.2, C5.1, R10.2, R3.2, R4.2, R5.2, R6.2, R7.2, R8.2, U6.5 (~{E1}), U6.8 (GND), U7.1 (VSS), U9.15 (GND); no longer C3.1 (Pin_1), J2.2, R9.5 (~{E1}), R9.8 (GND)
- net PB0: now also D1.2 (A), U7.10 (PB0); no longer U8.10 (PB0)
- net PB1: now also D2.2 (A), U7.11 (PB1); no longer U8.11 (PB1)
- net PB2: now also D3.2 (A), U7.12 (PB2); no longer U8.12 (PB2)
- net PB3: now also D4.2 (A), U7.13 (PB3); no longer U8.13 (PB3)
- net PB4: now also D5.2 (A), U7.14 (PB4); no longer U8.14 (PB4)
- net PB5: now also D6.2 (A), U7.15 (PB5); no longer U8.15 (PB5)
- net PB6: now also D7.2 (A), U7.16 (PB6); no longer U8.16 (PB6)
- net PB7: now also D8.2 (A), U7.17 (PB7); no longer U8.17 (PB7)
- net PHI2: now also U8.27 (PHI2), U7.25 (PHI2); no longer U8.25 (PHI2)
- net R/~{W}: now also U8.28 (R/~{W}), U7.22 (R/~{W}); no longer U8.22 (R/~{W})
- net VCC: now also U8.15 (VDD), X2.8 (Vcc), U6.16 (VCC), U6.6 (E2), U7.20 (VDD), U7.24 (CS1), U9.16 (VCC); no longer J2.1, R9.16 (VCC), R9.6 (E2), U8.20 (VDD), U8.24 (CS1)
- net ~{ACIA_CS}: now also U8.3 (~{CS1}), U6.11 (~{Y4}); no longer R9.11 (~{Y4})
- net ~{ACIA_RTS}: now also U8.8 (~{RTS}), U9.10 (T2IN); no longer C3.2 (Pin_2)
- net ~{IOSEL}: now also U6.4 (~{E0}); no longer R9.4 (~{E0})
- net ~{IRQ}: now also U8.26 (~{IRQ}), U7.21 (~{IRQ})
- net ~{RES}: now also U8.4 (~{RES}), U7.34 (~{RES}); no longer U8.34 (~{RES})
- net ~{VIA_CS}: now also U6.15 (~{Y0}), U7.23 (~{CS2}); no longer R9.15 (~{Y0}), U8.23 (~{CS2})
- removed net CA1: U8.40 (CA1), X2.9 (Pin_9)
- removed net CA2: U8.39 (CA2), X2.10 (Pin_10)
- removed net PA1: U8.3 (PA1), X2.2 (Pin_2)
- removed net PA2: U8.4 (PA2), X2.3 (Pin_3)
- net PA3: no longer names the net of U8.5 (RxC)
- net PA3: no longer X2.4 (Pin_4)
- net PA4 renamed ACIA_CLK
- net PA5: no longer names the net of U8.7 (XTLO)
- net PA5: no longer X2.6 (Pin_6)
- removed net PA6: U8.8 (PA6), X2.7 (Pin_7)
- removed net PA7: U8.9 (PA7), X2.8 (Pin_8)
- net XTLI: no longer names the net of C2.1
- net XTLI: now also U9.1 (C1+)
- net XTLO: no longer names the net of C2.2
- net XTLO: now also U9.3 (C1-)
- new net: D7.1 (K), R9.1
- new net: D2.1 (K), R4.1
- new net: D4.1 (K), R6.1
- new net: D8.1 (K), R10.1
- new net: D5.1 (K), R7.1
- new net: C3.1, U9.4 (C2+)
- new net: C3.2, U9.5 (C2-)
- new net: D3.1 (K), R5.1
- new net: D1.1 (K), R3.1
- new net: D6.1 (K), R8.1
- new net MAX232_VS+: C4.1, U9.2 (VS+)
- new net MAX232_VS-: C5.2, U9.6 (VS-)
- new net RS232_RTS: J2.8, U9.7 (T2OUT)
- new net RS232_RXD: J2.3, U9.13 (R1IN)
- new net RS232_TXD: J2.2, U9.14 (T1OUT)
- no-connect marks 10 -> 28
Other:
- note added: "1.8432 MHz oscillator drives XTLI. Pin 1 (EN) tied to +5V."
- note added: "I/O window $00:6000-$00:7FFF, 8 x 1 KB slots on A12:A11:A10 ~{Y0} $6000 VIA ~{Y4} $7000 ACIA ~{Y1} $6400 ~{Y2} $6800 ~{Y3} $6C00 ~{Y5} $7400 ~{Y6} $7800 ~{Y7} $7C00 (unallocated, not connected) ~{E1} (pin 5) is the reserved PHI2 hook: tie to ~{PHI2} to qualify the selects later (decode.pld NOTE 2). E2 (pin 6) is the active-high enable - it must be high."
- note added: "J2 DB9 female: 2 TxD (T1OUT), 3 RxD (R1IN), 8 RTS from ACIA (T2OUT), 5 GND. bios.s: 115200 8-N-1, flow control on ACIA ~{RTS}."
- note added: "MAX232N: T1 = ACIA TxD, R1 = ACIA RxD, T2 = ACIA ~{RTS}. R2IN and R2OUT not connected. C2-C5 1uF electrolytic; C4 from VS+ to GND, C5 from VS- to GND."
- note added: "Port A, CA1, CA2, CB1, CB2 not connected. IRQB is open drain on the W65C22N: wired straight to ~{IRQ} (pull-up R2, CPU sheet)."
- note added: "Port B LEDs: PBn -> LED -> resistor -> GND. R3-R10 values unknown."
- note added: "~{CTS}, ~{DSR}, ~{DCD} tied to GND. ~{DTR}, RxC and XTLO not connected."
- note removed: "D1 lets a W65C22S (totem-pole IRQB) share ~{IRQ} with the open-drain ACIA; also works with a W65C22N. Use a Schottky (< 0.5 V drop). Pull-up R3 is on the CPU sheet."
- note removed: "Decoupling: C8 U7, C9 U8, C10 U9."
- note removed: "I/O window $00:6000-$00:7FFF, 8 x 1 KB slots on A12:A11:A10 ~{Y0} $6000 VIA ~{Y4} $7000 ACIA ~{Y1} $6400 ~{Y2} $6800 ~{Y3} $6C00 ~{Y5} $7400 ~{Y6} $7800 ~{Y7} $7C00 (unallocated) ~{E1} (pin 5) is the reserved PHI2 hook: tie to ~{PHI2} to qualify the selects later (decode.pld NOTE 2). E2 (pin 6) is the active-high enable - it must be high."
- note removed: "J4: FTDI-style 6-pin TTL serial header 1 GND 2 CTS# (from ACIA ~{RTS}) 3 VCC (n/c) 4 TXD (to ACIA RxD) 5 RXD (from ACIA TxD) 6 RTS# (n/c) bios.s: 115200 8-N-1, flow control by toggling ACIA ~{RTS}. ~{CTS}, ~{DSR}, ~{DCD} tied low so the ACIA always transmits."
- note removed: "W65C22S ports have no current limiting: add series resistors when driving LEDs or an HD44780."
- title: I/O: '138 slot decoder, VIA, ACIA -> I/O: '138 slot decoder, VIA, ACIA, RS-232
- moved on the sheet: C2

Commit message: Show resistors R1-R10 as 1k (estimated)
The markings are unreadable; 1k is the builder's estimate and is noted
as such on the sheets and in kicad/README.md. Also list the unconnected
DB9 pins explicitly.

Co-Authored-By: Claude Opus 5.5 <noreply@anthropic.com>
Claude-Session: https://claude.ai/code/session_01GgTWzZQQJPzWrEMiSDZH6j
Parts:
- R10, R3, R4, R5, R6, R7, R8, R9: value ? -> 1k
Other:
- note added: "Port B LEDs: PBn -> LED -> resistor -> GND. R3-R10: 1k (estimated; markings unreadable)."
- note removed: "Port B LEDs: PBn -> LED -> resistor -> GND. R3-R10 values unknown."

Commit message: Mark R1-R10 as measured 1k
Co-Authored-By: Claude Opus 5.5 <noreply@anthropic.com>
Claude-Session: https://claude.ai/code/session_01GgTWzZQQJPzWrEMiSDZH6j
Other:
- note added: "Port B LEDs: PBn -> LED -> resistor -> GND. R3-R10: 1k (measured)."
- note removed: "Port B LEDs: PBn -> LED -> resistor -> GND. R3-R10: 1k (estimated; markings unreadable)."
Changed lines of the file:
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@@
 (wire (pts (xy 231.14 171.45) (xy 231.14 175.26)) (stroke (width 0) (type default)))
 (symbol (lib_id "be6502:GND") (at 231.14 182.88 0) (unit 1) (in_bom no) (on_board no) (dnp no) (property "Reference" "#PWR033" (at 231.14 189.23 0) (effects (font (size 1.27 1.27)) hide)) (property "Value" "GND" (at 231.14 186.69 0) (effects (font (size 1.27 1.27)))) (property "Footprint" "" (at 231.14 182.88 0) (effects (font (size 1.27 1.27)) hide)) (property "Datasheet" "" (at 231.14 182.88 0) (effects (font (size 1.27 1.27)) hide)) (pin "1") (instances (project "be6502" (path "/c8451a90-6bbf-595d-a4c9-ea2cdd0996a1/b62cf215-31ca-5406-b0ac-3a24a3937287" (reference "#PWR033") (unit 1)))))
-(text "Port B LEDs: PBn -> LED -> resistor -> GND.\nR3-R10: 1k (estimated; markings unreadable)." (at 157.48 200.66 0) (effects (font (size 1.27 1.27)) (justify left top)))
+(text "Port B LEDs: PBn -> LED -> resistor -> GND.\nR3-R10: 1k (measured)." (at 157.48 200.66 0) (effects (font (size 1.27 1.27)) (justify left top)))
 (symbol (lib_id "be6502:W65C51N") (at 279.4 101.6 0) (unit 1) (in_bom yes) (on_board yes) (dnp no) (property "Reference" "U8" (at 266.7 74.93 0) (effects (font (size 1.27 1.27)) (justify left bottom))) (property "Value" "W65C51N" (at 276.86 128.27 0) (effects (font (size 1.27 1.27)) (justify right top))) (property "Footprint" "Package_DIP:DIP-28_W15.24mm" (at 279.4 132.08 0) (effects (font (size 1.27 1.27)) hide)) (property "Datasheet" "https://www.westerndesigncenter.com/wdc/documentation/w65c51n.pdf" (at 279.4 134.62 0) (effects (font (size 1.27 1.27)) hide)) (pin "2") (pin "18") (pin "19") (pin "20") (pin "21") (pin "22") (pin "23") (pin "24") (pin "25") (pin "13") (pin "14") (pin "28") (pin "27") (pin "3") (pin "4") (pin "26") (pin "10") (pin "12") (pin "8") (pin "11") (pin "6") (pin "7") (pin "5") (pin "9") (pin "17") (pin "16") (pin "15") (pin "1") (instances (project "be6502" (path "/c8451a90-6bbf-595d-a4c9-ea2cdd0996a1/b62cf215-31ca-5406-b0ac-3a24a3937287" (reference "U8") (unit 1)))))
 (wire (pts (xy 261.62 106.68) (xy 256.54 106.68)) (stroke (width 0) (type default)))

Commit message: Add a two-layer PCB layout made from the schematic
Assign footprints to the passives, LEDs, switch and connectors, place
all parts on a 175 x 125 mm board, route it with a small grid router,
and pour GND on both layers. DRC in KiCad 7.0.11 reports no violations
and no unconnected pads. Renders and the generating scripts are included.

Co-Authored-By: Claude Opus 5.5 <noreply@anthropic.com>
Claude-Session: https://claude.ai/code/session_01PBQiX4PgHFxHybqnr7fDuN
Parts:
- C2, C3, C4, C5: footprint (none) -> Capacitor_THT:CP_Radial_D5.0mm_P2.00mm
- D1, D2, D3, D4, D5, D6, D7, D8: footprint (none) -> LED_THT:LED_D3.0mm
- J2: footprint (none) -> Connector_Dsub:DSUB-9_Female_Horizontal_P2.77x2.84mm_EdgePinOffset7.70mm_Housed_MountingHolesOffset9.12mm
- R10, R3, R4, R5, R6, R7, R8, R9: footprint (none) -> Resistor_THT:R_Axial_DIN0207_L6.3mm_D2.5mm_P7.62mm_Horizontal
