File: kicad/expansion.kicad_sch (KiCad schematic)
At the start: 19 parts, among them J3 EXPANSION, J4 VIA PORTS, J5 EXT CLOCK, U10 74ACT08

Commit message: Add 4-layer PCB with all parts placed (unrouted)
190 x 120 mm, F.Cu / In1 GND plane / In2 +5V plane / B.Cu. Every
footprint carries its nets and is linked to its schematic symbol
(0 schematic-parity issues), so Update PCB from Schematic works in
place. Power and Default net classes are in the project file.

Placement: expansion header on the left edge next to the CPU; power,
switch and reset along the top; memory and I/O across the middle; VIA
header and DB9 on the right edge; LEDs and test points along the bottom;
100nF decoupling at each IC; M3 holes in the corners.

DRC: no courtyard, clearance or hole violations; only unrouted
connections and the DB9 shell silkscreen overhanging the edge.

Mounting-hole symbols are now excluded from the BOM to match their
footprints.

Co-Authored-By: Claude Opus 5.5 <noreply@anthropic.com>
Claude-Session: https://claude.ai/code/session_01WF6ESyzfg6uQED2DRD2W4Z
Parts:
- H1, H2, H3, H4: now left out of the parts list
Changed lines of the file:
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@@
 (global_label "~{IRQ}" (shape passive) (at 350.52 218.44 270) (fields_autoplaced) (effects (font (size 1.27 1.27)) (justify right)) (property "Intersheetrefs" "${INTERSHEET_REFS}" (at 350.52 218.44 0) (effects (font (size 1.27 1.27)) (justify right) hide)))
 (text "Test points: +5V, two GND loops for scope grounds, PHI2,\nCLK2, ~{RES}, ~{IRQ}.  The full bus is also on J3 for a\nlogic analyzer or an Arduino bus monitor." (at 266.7 233.68 0) (effects (font (size 1.27 1.27)) (justify left top)))
-(symbol (lib_id "be6502:MountingHole") (at 203.2 254 0) (unit 1) (in_bom yes) (on_board yes) (dnp no) (property "Reference" "H1" (at 203.2 250.19 0) (effects (font (size 1.27 1.27)))) (property "Value" "M3" (at 203.2 257.81 0) (effects (font (size 1.27 1.27)))) (property "Footprint" "MountingHole:MountingHole_3.2mm_M3" (at 203.2 254 0) (effects (font (size 1.27 1.27)) hide)) (property "Datasheet" "" (at 203.2 254 0) (effects (font (size 1.27 1.27)) hide))  (instances (project "be6502" (path "/c8451a90-6bbf-595d-a4c9-ea2cdd0996a1/55b79aa4-89f4-5549-b0fa-20da30c1af54" (reference "H1") (unit 1)))))
-(symbol (lib_id "be6502:MountingHole") (at 215.9 254 0) (unit 1) (in_bom yes) (on_board yes) (dnp no) (property "Reference" "H2" (at 215.9 250.19 0) (effects (font (size 1.27 1.27)))) (property "Value" "M3" (at 215.9 257.81 0) (effects (font (size 1.27 1.27)))) (property "Footprint" "MountingHole:MountingHole_3.2mm_M3" (at 215.9 254 0) (effects (font (size 1.27 1.27)) hide)) (property "Datasheet" "" (at 215.9 254 0) (effects (font (size 1.27 1.27)) hide))  (instances (project "be6502" (path "/c8451a90-6bbf-595d-a4c9-ea2cdd0996a1/55b79aa4-89f4-5549-b0fa-20da30c1af54" (reference "H2") (unit 1)))))
-(symbol (lib_id "be6502:MountingHole") (at 228.6 254 0) (unit 1) (in_bom yes) (on_board yes) (dnp no) (property "Reference" "H3" (at 228.6 250.19 0) (effects (font (size 1.27 1.27)))) (property "Value" "M3" (at 228.6 257.81 0) (effects (font (size 1.27 1.27)))) (property "Footprint" "MountingHole:MountingHole_3.2mm_M3" (at 228.6 254 0) (effects (font (size 1.27 1.27)) hide)) (property "Datasheet" "" (at 228.6 254 0) (effects (font (size 1.27 1.27)) hide))  (instances (project "be6502" (path "/c8451a90-6bbf-595d-a4c9-ea2cdd0996a1/55b79aa4-89f4-5549-b0fa-20da30c1af54" (reference "H3") (unit 1)))))
-(symbol (lib_id "be6502:MountingHole") (at 241.3 254 0) (unit 1) (in_bom yes) (on_board yes) (dnp no) (property "Reference" "H4" (at 241.3 250.19 0) (effects (font (size 1.27 1.27)))) (property "Value" "M3" (at 241.3 257.81 0) (effects (font (size 1.27 1.27)))) (property "Footprint" "MountingHole:MountingHole_3.2mm_M3" (at 241.3 254 0) (effects (font (size 1.27 1.27)) hide)) (property "Datasheet" "" (at 241.3 254 0) (effects (font (size 1.27 1.27)) hide))  (instances (project "be6502" (path "/c8451a90-6bbf-595d-a4c9-ea2cdd0996a1/55b79aa4-89f4-5549-b0fa-20da30c1af54" (reference "H4") (unit 1)))))
+(symbol (lib_id "be6502:MountingHole") (at 203.2 254 0) (unit 1) (in_bom no) (on_board yes) (dnp no) (property "Reference" "H1" (at 203.2 250.19 0) (effects (font (size 1.27 1.27)))) (property "Value" "M3" (at 203.2 257.81 0) (effects (font (size 1.27 1.27)))) (property "Footprint" "MountingHole:MountingHole_3.2mm_M3" (at 203.2 254 0) (effects (font (size 1.27 1.27)) hide)) (property "Datasheet" "" (at 203.2 254 0) (effects (font (size 1.27 1.27)) hide))  (instances (project "be6502" (path "/c8451a90-6bbf-595d-a4c9-ea2cdd0996a1/55b79aa4-89f4-5549-b0fa-20da30c1af54" (reference "H1") (unit 1)))))
+(symbol (lib_id "be6502:MountingHole") (at 215.9 254 0) (unit 1) (in_bom no) (on_board yes) (dnp no) (property "Reference" "H2" (at 215.9 250.19 0) (effects (font (size 1.27 1.27)))) (property "Value" "M3" (at 215.9 257.81 0) (effects (font (size 1.27 1.27)))) (property "Footprint" "MountingHole:MountingHole_3.2mm_M3" (at 215.9 254 0) (effects (font (size 1.27 1.27)) hide)) (property "Datasheet" "" (at 215.9 254 0) (effects (font (size 1.27 1.27)) hide))  (instances (project "be6502" (path "/c8451a90-6bbf-595d-a4c9-ea2cdd0996a1/55b79aa4-89f4-5549-b0fa-20da30c1af54" (reference "H2") (unit 1)))))
+(symbol (lib_id "be6502:MountingHole") (at 228.6 254 0) (unit 1) (in_bom no) (on_board yes) (dnp no) (property "Reference" "H3" (at 228.6 250.19 0) (effects (font (size 1.27 1.27)))) (property "Value" "M3" (at 228.6 257.81 0) (effects (font (size 1.27 1.27)))) (property "Footprint" "MountingHole:MountingHole_3.2mm_M3" (at 228.6 254 0) (effects (font (size 1.27 1.27)) hide)) (property "Datasheet" "" (at 228.6 254 0) (effects (font (size 1.27 1.27)) hide))  (instances (project "be6502" (path "/c8451a90-6bbf-595d-a4c9-ea2cdd0996a1/55b79aa4-89f4-5549-b0fa-20da30c1af54" (reference "H3") (unit 1)))))
+(symbol (lib_id "be6502:MountingHole") (at 241.3 254 0) (unit 1) (in_bom no) (on_board yes) (dnp no) (property "Reference" "H4" (at 241.3 250.19 0) (effects (font (size 1.27 1.27)))) (property "Value" "M3" (at 241.3 257.81 0) (effects (font (size 1.27 1.27)))) (property "Footprint" "MountingHole:MountingHole_3.2mm_M3" (at 241.3 254 0) (effects (font (size 1.27 1.27)) hide)) (property "Datasheet" "" (at 241.3 254 0) (effects (font (size 1.27 1.27)) hide))  (instances (project "be6502" (path "/c8451a90-6bbf-595d-a4c9-ea2cdd0996a1/55b79aa4-89f4-5549-b0fa-20da30c1af54" (reference "H4") (unit 1)))))
 )
