File: kicad/cpu.kicad_sch (KiCad schematic)
At the start: 7 parts, among them SW1 RESET, U1 W65C816S, U2 74HC573, U3 ATF22V10C 816DEC02, X1 12MHz

Commit message: Add a two-layer PCB layout made from the schematic
Assign footprints to the passives, LEDs, switch and connectors, place
all parts on a 175 x 125 mm board, route it with a small grid router,
and pour GND on both layers. DRC in KiCad 7.0.11 reports no violations
and no unconnected pads. Renders and the generating scripts are included.

Co-Authored-By: Claude Opus 5.5 <noreply@anthropic.com>
Claude-Session: https://claude.ai/code/session_01PBQiX4PgHFxHybqnr7fDuN
Parts:
- R1, R2: footprint (none) -> Resistor_THT:R_Axial_DIN0207_L6.3mm_D2.5mm_P7.62mm_Horizontal
- SW1: footprint (none) -> Button_Switch_THT:SW_PUSH_6mm
Changed lines of the file:
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@@
 (symbol (lib_id "be6502:GND") (at 309.88 60.96 0) (unit 1) (in_bom no) (on_board no) (dnp no) (property "Reference" "#PWR010" (at 309.88 67.31 0) (effects (font (size 1.27 1.27)) hide)) (property "Value" "GND" (at 309.88 64.77 0) (effects (font (size 1.27 1.27)))) (property "Footprint" "" (at 309.88 60.96 0) (effects (font (size 1.27 1.27)) hide)) (property "Datasheet" "" (at 309.88 60.96 0) (effects (font (size 1.27 1.27)) hide)) (pin "1") (instances (project "be6502" (path "/c8451a90-6bbf-595d-a4c9-ea2cdd0996a1/f67db34f-3d17-54e5-a1b6-ae57793ddc10" (reference "#PWR010") (unit 1)))))
 (text "12 MHz oscillator, 2x PHI2.  U3 divides it\nby two to make PHI2 = 6 MHz.  Pin 1 not connected." (at 292.1 66.04 0) (effects (font (size 1.27 1.27)) (justify left top)))
-(symbol (lib_id "be6502:R") (at 304.8 99.06 0) (unit 1) (in_bom yes) (on_board yes) (dnp no) (property "Reference" "R1" (at 306.832 99.06 90) (effects (font (size 1.27 1.27)))) (property "Value" "1k" (at 304.8 99.06 90) (effects (font (size 1.27 1.27)))) (property "Footprint" "" (at 303.022 99.06 90) (effects (font (size 1.27 1.27)) hide)) (property "Datasheet" "~" (at 304.8 99.06 0) (effects (font (size 1.27 1.27)) hide)) (pin "1") (pin "2") (instances (project "be6502" (path "/c8451a90-6bbf-595d-a4c9-ea2cdd0996a1/f67db34f-3d17-54e5-a1b6-ae57793ddc10" (reference "R1") (unit 1)))))
+(symbol (lib_id "be6502:R") (at 304.8 99.06 0) (unit 1) (in_bom yes) (on_board yes) (dnp no) (property "Reference" "R1" (at 306.832 99.06 90) (effects (font (size 1.27 1.27)))) (property "Value" "1k" (at 304.8 99.06 90) (effects (font (size 1.27 1.27)))) (property "Footprint" "Resistor_THT:R_Axial_DIN0207_L6.3mm_D2.5mm_P7.62mm_Horizontal" (at 303.022 99.06 90) (effects (font (size 1.27 1.27)) hide)) (property "Datasheet" "~" (at 304.8 99.06 0) (effects (font (size 1.27 1.27)) hide)) (pin "1") (pin "2") (instances (project "be6502" (path "/c8451a90-6bbf-595d-a4c9-ea2cdd0996a1/f67db34f-3d17-54e5-a1b6-ae57793ddc10" (reference "R1") (unit 1)))))
 (wire (pts (xy 304.8 95.25) (xy 304.8 92.71)) (stroke (width 0) (type default)))
 (symbol (lib_id "be6502:VCC") (at 304.8 92.71 0) (unit 1) (in_bom no) (on_board no) (dnp no) (property "Reference" "#PWR011" (at 304.8 96.52 0) (effects (font (size 1.27 1.27)) hide)) (property "Value" "VCC" (at 304.8 88.9 0) (effects (font (size 1.27 1.27)))) (property "Footprint" "" (at 304.8 92.71 0) (effects (font (size 1.27 1.27)) hide)) (property "Datasheet" "" (at 304.8 92.71 0) (effects (font (size 1.27 1.27)) hide)) (pin "1") (instances (project "be6502" (path "/c8451a90-6bbf-595d-a4c9-ea2cdd0996a1/f67db34f-3d17-54e5-a1b6-ae57793ddc10" (reference "#PWR011") (unit 1)))))
 (wire (pts (xy 304.8 102.87) (xy 304.8 107.95)) (stroke (width 0) (type default)))
 (global_label "~{RES}" (shape output) (at 304.8 107.95 270) (fields_autoplaced) (effects (font (size 1.27 1.27)) (justify right)) (property "Intersheetrefs" "${INTERSHEET_REFS}" (at 304.8 107.95 0) (effects (font (size 1.27 1.27)) (justify right) hide)))
-(symbol (lib_id "be6502:SW_Push") (at 327.66 116.84 0) (unit 1) (in_bom yes) (on_board yes) (dnp no) (property "Reference" "SW1" (at 328.93 114.3 0) (effects (font (size 1.27 1.27)) (justify left))) (property "Value" "RESET" (at 327.66 118.364 0) (effects (font (size 1.27 1.27)))) (property "Footprint" "" (at 327.66 111.76 0) (effects (font (size 1.27 1.27)) hide)) (property "Datasheet" "~" (at 327.66 111.76 0) (effects (font (size 1.27 1.27)) hide)) (pin "1") (pin "2") (instances (project "be6502" (path "/c8451a90-6bbf-595d-a4c9-ea2cdd0996a1/f67db34f-3d17-54e5-a1b6-ae57793ddc10" (reference "SW1") (unit 1)))))
+(symbol (lib_id "be6502:SW_Push") (at 327.66 116.84 0) (unit 1) (in_bom yes) (on_board yes) (dnp no) (property "Reference" "SW1" (at 328.93 114.3 0) (effects (font (size 1.27 1.27)) (justify left))) (property "Value" "RESET" (at 327.66 118.364 0) (effects (font (size 1.27 1.27)))) (property "Footprint" "Button_Switch_THT:SW_PUSH_6mm" (at 327.66 111.76 0) (effects (font (size 1.27 1.27)) hide)) (property "Datasheet" "~" (at 327.66 111.76 0) (effects (font (size 1.27 1.27)) hide)) (pin "1") (pin "2") (instances (project "be6502" (path "/c8451a90-6bbf-595d-a4c9-ea2cdd0996a1/f67db34f-3d17-54e5-a1b6-ae57793ddc10" (reference "SW1") (unit 1)))))
 (wire (pts (xy 322.58 116.84) (xy 317.5 116.84)) (stroke (width 0) (type default)))
 (global_label "~{RES}" (shape output) (at 317.5 116.84 180) (fields_autoplaced) (effects (font (size 1.27 1.27)) (justify right)) (property "Intersheetrefs" "${INTERSHEET_REFS}" (at 317.5 116.84 0) (effects (font (size 1.27 1.27)) (justify right) hide)))
 (wire (pts (xy 332.74 116.84) (xy 335.28 116.84)) (stroke (width 0) (type default)))
 (symbol (lib_id "be6502:GND") (at 335.28 116.84 0) (unit 1) (in_bom no) (on_board no) (dnp no) (property "Reference" "#PWR012" (at 335.28 123.19 0) (effects (font (size 1.27 1.27)) hide)) (property "Value" "GND" (at 335.28 120.65 0) (effects (font (size 1.27 1.27)))) (property "Footprint" "" (at 335.28 116.84 0) (effects (font (size 1.27 1.27)) hide)) (property "Datasheet" "" (at 335.28 116.84 0) (effects (font (size 1.27 1.27)) hide)) (pin "1") (instances (project "be6502" (path "/c8451a90-6bbf-595d-a4c9-ea2cdd0996a1/f67db34f-3d17-54e5-a1b6-ae57793ddc10" (reference "#PWR012") (unit 1)))))
-(symbol (lib_id "be6502:R") (at 304.8 154.94 0) (unit 1) (in_bom yes) (on_board yes) (dnp no) (property "Reference" "R2" (at 306.832 154.94 90) (effects (font (size 1.27 1.27)))) (property "Value" "1k" (at 304.8 154.94 90) (effects (font (size 1.27 1.27)))) (property "Footprint" "" (at 303.022 154.94 90) (effects (font (size 1.27 1.27)) hide)) (property "Datasheet" "~" (at 304.8 154.94 0) (effects (font (size 1.27 1.27)) hide)) (pin "1") (pin "2") (instances (project "be6502" (path "/c8451a90-6bbf-595d-a4c9-ea2cdd0996a1/f67db34f-3d17-54e5-a1b6-ae57793ddc10" (reference "R2") (unit 1)))))
+(symbol (lib_id "be6502:R") (at 304.8 154.94 0) (unit 1) (in_bom yes) (on_board yes) (dnp no) (property "Reference" "R2" (at 306.832 154.94 90) (effects (font (size 1.27 1.27)))) (property "Value" "1k" (at 304.8 154.94 90) (effects (font (size 1.27 1.27)))) (property "Footprint" "Resistor_THT:R_Axial_DIN0207_L6.3mm_D2.5mm_P7.62mm_Horizontal" (at 303.022 154.94 90) (effects (font (size 1.27 1.27)) hide)) (property "Datasheet" "~" (at 304.8 154.94 0) (effects (font (size 1.27 1.27)) hide)) (pin "1") (pin "2") (instances (project "be6502" (path "/c8451a90-6bbf-595d-a4c9-ea2cdd0996a1/f67db34f-3d17-54e5-a1b6-ae57793ddc10" (reference "R2") (unit 1)))))
 (wire (pts (xy 304.8 151.13) (xy 304.8 148.59)) (stroke (width 0) (type default)))
 (symbol (lib_id "be6502:VCC") (at 304.8 148.59 0) (unit 1) (in_bom no) (on_board no) (dnp no) (property "Reference" "#PWR013" (at 304.8 152.4 0) (effects (font (size 1.27 1.27)) hide)) (property "Value" "VCC" (at 304.8 144.78 0) (effects (font (size 1.27 1.27)))) (property "Footprint" "" (at 304.8 148.59 0) (effects (font (size 1.27 1.27)) hide)) (property "Datasheet" "" (at 304.8 148.59 0) (effects (font (size 1.27 1.27)) hide)) (pin "1") (instances (project "be6502" (path "/c8451a90-6bbf-595d-a4c9-ea2cdd0996a1/f67db34f-3d17-54e5-a1b6-ae57793ddc10" (reference "#PWR013") (unit 1)))))
