File: kicad/power.kicad_sch (KiCad schematic)
At the start: 2 parts, among them J1 BENCH SUPPLY +5V

Commit message: Add a two-layer PCB layout made from the schematic
Assign footprints to the passives, LEDs, switch and connectors, place
all parts on a 175 x 125 mm board, route it with a small grid router,
and pour GND on both layers. DRC in KiCad 7.0.11 reports no violations
and no unconnected pads. Renders and the generating scripts are included.

Co-Authored-By: Claude Opus 5.5 <noreply@anthropic.com>
Claude-Session: https://claude.ai/code/session_01PBQiX4PgHFxHybqnr7fDuN
Parts:
- C1: footprint (none) -> Capacitor_THT:CP_Radial_D5.0mm_P2.00mm
- J1: footprint (none) -> TerminalBlock_Phoenix:TerminalBlock_Phoenix_MKDS-1,5-2-5.08_1x02_P5.08mm_Horizontal
Changed lines of the file:
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@@
 (paper "A4")
 (title_block (title "Power") (date "2026-10-16") (rev "1") (company "be6502") (comment 1 "W65C816S breadboard computer - see README.md and pld/decode.pld") (comment 2 "Active-low signals use KiCad overbar notation, e.g. ~{IOSEL}"))
-(symbol (lib_id "be6502:Conn_01x02") (at 76.2 76.2 0) (unit 1) (in_bom yes) (on_board yes) (dnp no) (property "Reference" "J1" (at 76.2 73.66 0) (effects (font (size 1.27 1.27)))) (property "Value" "BENCH SUPPLY +5V" (at 76.2 81.28 0) (effects (font (size 1.27 1.27)))) (property "Footprint" "" (at 76.2 76.2 0) (effects (font (size 1.27 1.27)) hide)) (property "Datasheet" "~" (at 76.2 76.2 0) (effects (font (size 1.27 1.27)) hide)) (pin "1") (pin "2") (instances (project "be6502" (path "/c8451a90-6bbf-595d-a4c9-ea2cdd0996a1/b455a6f5-8f62-5a1c-b7d1-ce7f0c9edb4a" (reference "J1") (unit 1)))))
+(symbol (lib_id "be6502:Conn_01x02") (at 76.2 76.2 0) (unit 1) (in_bom yes) (on_board yes) (dnp no) (property "Reference" "J1" (at 76.2 73.66 0) (effects (font (size 1.27 1.27)))) (property "Value" "BENCH SUPPLY +5V" (at 76.2 81.28 0) (effects (font (size 1.27 1.27)))) (property "Footprint" "TerminalBlock_Phoenix:TerminalBlock_Phoenix_MKDS-1,5-2-5.08_1x02_P5.08mm_Horizontal" (at 76.2 76.2 0) (effects (font (size 1.27 1.27)) hide)) (property "Datasheet" "~" (at 76.2 76.2 0) (effects (font (size 1.27 1.27)) hide)) (pin "1") (pin "2") (instances (project "be6502" (path "/c8451a90-6bbf-595d-a4c9-ea2cdd0996a1/b455a6f5-8f62-5a1c-b7d1-ce7f0c9edb4a" (reference "J1") (unit 1)))))
 (wire (pts (xy 71.12 76.2) (xy 58.42 76.2)) (stroke (width 0) (type default)))
 (wire (pts (xy 58.42 76.2) (xy 43.18 76.2)) (stroke (width 0) (type default)))
@@
 (symbol (lib_id "be6502:PWR_FLAG") (at 58.42 78.74 180) (unit 1) (in_bom no) (on_board no) (dnp no) (property "Reference" "#FLG02" (at 58.42 80.645 0) (effects (font (size 1.27 1.27)) hide)) (property "Value" "PWR_FLAG" (at 58.42 82.55 0) (effects (font (size 1.27 1.27)))) (property "Footprint" "" (at 58.42 78.74 0) (effects (font (size 1.27 1.27)) hide)) (property "Datasheet" "~" (at 58.42 78.74 0) (effects (font (size 1.27 1.27)) hide)) (pin "1") (instances (project "be6502" (path "/c8451a90-6bbf-595d-a4c9-ea2cdd0996a1/b455a6f5-8f62-5a1c-b7d1-ce7f0c9edb4a" (reference "#FLG02") (unit 1)))))
 (symbol (lib_id "be6502:GND") (at 43.18 83.82 0) (unit 1) (in_bom no) (on_board no) (dnp no) (property "Reference" "#PWR047" (at 43.18 90.17 0) (effects (font (size 1.27 1.27)) hide)) (property "Value" "GND" (at 43.18 87.63 0) (effects (font (size 1.27 1.27)))) (property "Footprint" "" (at 43.18 83.82 0) (effects (font (size 1.27 1.27)) hide)) (property "Datasheet" "" (at 43.18 83.82 0) (effects (font (size 1.27 1.27)) hide)) (pin "1") (instances (project "be6502" (path "/c8451a90-6bbf-595d-a4c9-ea2cdd0996a1/b455a6f5-8f62-5a1c-b7d1-ce7f0c9edb4a" (reference "#PWR047") (unit 1)))))
-(symbol (lib_id "be6502:C_Polarized") (at 101.6 78.74 0) (unit 1) (in_bom yes) (on_board yes) (dnp no) (property "Reference" "C1" (at 102.235 76.2 0) (effects (font (size 1.27 1.27)) (justify left))) (property "Value" "0.1uF" (at 102.235 81.28 0) (effects (font (size 1.27 1.27)) (justify left))) (property "Footprint" "" (at 102.5652 82.55 0) (effects (font (size 1.27 1.27)) hide)) (property "Datasheet" "~" (at 101.6 78.74 0) (effects (font (size 1.27 1.27)) hide)) (pin "1") (pin "2") (instances (project "be6502" (path "/c8451a90-6bbf-595d-a4c9-ea2cdd0996a1/b455a6f5-8f62-5a1c-b7d1-ce7f0c9edb4a" (reference "C1") (unit 1)))))
+(symbol (lib_id "be6502:C_Polarized") (at 101.6 78.74 0) (unit 1) (in_bom yes) (on_board yes) (dnp no) (property "Reference" "C1" (at 102.235 76.2 0) (effects (font (size 1.27 1.27)) (justify left))) (property "Value" "0.1uF" (at 102.235 81.28 0) (effects (font (size 1.27 1.27)) (justify left))) (property "Footprint" "Capacitor_THT:CP_Radial_D5.0mm_P2.00mm" (at 102.5652 82.55 0) (effects (font (size 1.27 1.27)) hide)) (property "Datasheet" "~" (at 101.6 78.74 0) (effects (font (size 1.27 1.27)) hide)) (pin "1") (pin "2") (instances (project "be6502" (path "/c8451a90-6bbf-595d-a4c9-ea2cdd0996a1/b455a6f5-8f62-5a1c-b7d1-ce7f0c9edb4a" (reference "C1") (unit 1)))))
 (symbol (lib_id "be6502:VCC") (at 101.6 74.93 0) (unit 1) (in_bom no) (on_board no) (dnp no) (property "Reference" "#PWR048" (at 101.6 78.74 0) (effects (font (size 1.27 1.27)) hide)) (property "Value" "VCC" (at 101.6 71.12 0) (effects (font (size 1.27 1.27)))) (property "Footprint" "" (at 101.6 74.93 0) (effects (font (size 1.27 1.27)) hide)) (property "Datasheet" "" (at 101.6 74.93 0) (effects (font (size 1.27 1.27)) hide)) (pin "1") (instances (project "be6502" (path "/c8451a90-6bbf-595d-a4c9-ea2cdd0996a1/b455a6f5-8f62-5a1c-b7d1-ce7f0c9edb4a" (reference "#PWR048") (unit 1)))))
 (symbol (lib_id "be6502:GND") (at 101.6 82.55 0) (unit 1) (in_bom no) (on_board no) (dnp no) (property "Reference" "#PWR049" (at 101.6 88.9 0) (effects (font (size 1.27 1.27)) hide)) (property "Value" "GND" (at 101.6 86.36 0) (effects (font (size 1.27 1.27)))) (property "Footprint" "" (at 101.6 82.55 0) (effects (font (size 1.27 1.27)) hide)) (property "Datasheet" "" (at 101.6 82.55 0) (effects (font (size 1.27 1.27)) hide)) (pin "1") (instances (project "be6502" (path "/c8451a90-6bbf-595d-a4c9-ea2cdd0996a1/b455a6f5-8f62-5a1c-b7d1-ce7f0c9edb4a" (reference "#PWR049") (unit 1)))))
